Commit message: Fix xtion_pro_live mesh paths

File: urdf/camera/orbbec_astra.urdf.xacro (robot description, xacro)
@@ -35,5 +35,5 @@
         <origin xyz="0 0 0" rpy="0 0 0"/>
         <geometry>
-          <mesh filename="file://$(find tiago_description)/meshes/camera/xtion_pro_live/xtion_pro_live.dae" />
+          <mesh filename="file://$(find pal_urdf_utils)/meshes/camera/xtion_pro_live.dae" />
         </geometry>
         <material name="Grey">

File: urdf/camera/xtion_pro_live.urdf.xacro (robot description, xacro)
@@ -34,5 +34,5 @@
         <origin xyz="0 0 0" rpy="0 0 0"/>
         <geometry>
-          <mesh filename="file://$(find tiago_description)/meshes/camera/xtion_pro_live/xtion_pro_live.dae" />
+          <mesh filename="file://$(find pal_urdf_utils)/meshes/camera/xtion_pro_live.dae" />
         </geometry>
         <material name="Grey">
