Commit message: avoid duplicate definition of the camera config

File: urdf/camera/structure_sensor.gazebo.xacro (robot description, xacro)
@@ -14,10 +14,20 @@
 <robot xmlns:xacro="http://ros.org/wiki/xacro">
   <xacro:macro name="structure_sensor_rgbd_camera_gazebo" params="name">
+    <xacro:if value="${gazebo_version == 'classic'}">
+      <xacro:property name="camera_type" value="depth"/>
+    </xacro:if>
+    <xacro:if value="${gazebo_version == 'gazebo'}">
+      <xacro:property name="camera_type" value="rgbd_camera"/>
+    </xacro:if>
     <gazebo reference="${name}_link">
       <!-- IR + depth -->
-      <xacro:if value="${gazebo_version == 'classic'}">
-        <sensor type="depth" name="${name}_frame_sensor">
+        <sensor type="${camera_type}" name="${name}_frame_sensor">
           <always_on>true</always_on>
           <update_rate>6.0</update_rate>
+          <gz_frame_id>${name}_optical_frame</gz_frame_id>
+          <always_on>1</always_on>
+          <update_rate>10</update_rate>
+          <visualize>0</visualize>
+          <topic>${name}</topic>
           <camera>
             <horizontal_fov>${58.0 * deg_to_rad}</horizontal_fov>
@@ -39,117 +49,79 @@
             </distortion>
           </camera>
-          <plugin name="${name}_ir" filename="libgazebo_ros_camera.so">
-            <camera_name>${name}</camera_name>
-            <frame_name>${name}_optical_frame</frame_name>
-            <max_depth>10.0</max_depth>
-            <ros>
-              <namespace>${namespace}</namespace>
-              <remapping>${name}/image_raw:=${name}/ir/image_raw</remapping>
-              <remapping>${name}/camera_info:=${name}/ir/camera_info</remapping>
-              <remapping>${name}/image_raw/compressed:=${name}/ir/image_raw/compressed</remapping>
-              <remapping>${name}/image_raw/compressedDepth:=${name}/ir/image_raw/compressedDepth</remapping>
-              <remapping>${name}/image_raw/theora:=${name}/ir/image_raw/theora</remapping>
-              <remapping>${name}/points:=${name}/depth/points</remapping>
-              <qos>
-                <topic name="${name}/ir/image_raw">
-                  <publisher>
-                    <reliability>best_effort</reliability>
-                    <durability>volatile</durability>
-                    <history depth="1">keep_last</history>
-                    <liveliness>automatic</liveliness>
-                  </publisher>
-                </topic>
-                <topic name="${name}/ir/image_raw/compressed">
-                  <publisher>
-                    <reliability>best_effort</reliability>
-                    <durability>volatile</durability>
-                    <history depth="1">keep_last</history>
-                    <liveliness>automatic</liveliness>
-                  </publisher>
-                </topic>
-                <topic name="${name}/ir/image_raw/compressedDepth">
-                  <publisher>
-                    <reliability>best_effort</reliability>
-                    <durability>volatile</durability>
-                    <history depth="1">keep_last</history>
-                    <liveliness>automatic</liveliness>
-                  </publisher>
-                </topic>
-                <topic name="${name}/depth/image_raw">
-                  <publisher>
-                    <reliability>best_effort</reliability>
-                    <durability>volatile</durability>
-                    <history depth="1">keep_last</history>
-                    <liveliness>automatic</liveliness>
-                  </publisher>
-                </topic>
-                <topic name="${name}/depth/image_raw/compressed">
-                  <publisher>
-                    <reliability>best_effort</reliability>
-                    <durability>volatile</durability>
-                    <history depth="1">keep_last</history>
-                    <liveliness>automatic</liveliness>
-                  </publisher>
-                </topic>
-                <topic name="${name}/depth/image_raw/compressedDepth">
-                  <publisher>
-                    <reliability>best_effort</reliability>
-                    <durability>volatile</durability>
-                    <history depth="1">keep_last</history>
-                    <liveliness>automatic</liveliness>
-                  </publisher>
-                </topic>
-                <topic name="${name}/depth/points">
-                  <publisher>
-                    <reliability>best_effort</reliability>
-                    <durability>volatile</durability>
-                    <history depth="1">keep_last</history>
-                    <liveliness>automatic</liveliness>
-                  </publisher>
-                </topic>
-              </qos>
-            </ros>
-          </plugin>
+          <xacro:if value="${gazebo_version == 'classic'}">
+            <plugin name="${name}_ir" filename="libgazebo_ros_camera.so">
+              <camera_name>${name}</camera_name>
+              <frame_name>${name}_optical_frame</frame_name>
+              <max_depth>10.0</max_depth>
+              <ros>
+                <namespace>${namespace}</namespace>
+                <remapping>${name}/image_raw:=${name}/ir/image_raw</remapping>
+                <remapping>${name}/camera_info:=${name}/ir/camera_info</remapping>
+                <remapping>${name}/image_raw/compressed:=${name}/ir/image_raw/compressed</remapping>
+                <remapping>${name}/image_raw/compressedDepth:=${name}/ir/image_raw/compressedDepth</remapping>
+                <remapping>${name}/image_raw/theora:=${name}/ir/image_raw/theora</remapping>
+                <remapping>${name}/points:=${name}/depth/points</remapping>
+                <qos>
+                  <topic name="${name}/ir/image_raw">
+                    <publisher>
+                      <reliability>best_effort</reliability>
+                      <durability>volatile</durability>
+                      <history depth="1">keep_last</history>
+                      <liveliness>automatic</liveliness>
+                    </publisher>
+                  </topic>
+                  <topic name="${name}/ir/image_raw/compressed">
+                    <publisher>
+                      <reliability>best_effort</reliability>
+                      <durability>volatile</durability>
+                      <history depth="1">keep_last</history>
+                      <liveliness>automatic</liveliness>
+                    </publisher>
+                  </topic>
+                  <topic name="${name}/ir/image_raw/compressedDepth">
+                    <publisher>
+                      <reliability>best_effort</reliability>
+                      <durability>volatile</durability>
+                      <history depth="1">keep_last</history>
+                      <liveliness>automatic</liveliness>
+                    </publisher>
+                  </topic>
+                  <topic name="${name}/depth/image_raw">
+                    <publisher>
+                      <reliability>best_effort</reliability>
+                      <durability>volatile</durability>
+                      <history depth="1">keep_last</history>
+                      <liveliness>automatic</liveliness>
+                    </publisher>
+                  </topic>
+                  <topic name="${name}/depth/image_raw/compressed">
+                    <publisher>
+                      <reliability>best_effort</reliability>
+                      <durability>volatile</durability>
+                      <history depth="1">keep_last</history>
+                      <liveliness>automatic</liveliness>
+                    </publisher>
+                  </topic>
+                  <topic name="${name}/depth/image_raw/compressedDepth">
+                    <publisher>
+                      <reliability>best_effort</reliability>
+                      <durability>volatile</durability>
+                      <history depth="1">keep_last</history>
+                      <liveliness>automatic</liveliness>
+                    </publisher>
+                  </topic>
+                  <topic name="${name}/depth/points">
+                    <publisher>
+                      <reliability>best_effort</reliability>
+                      <durability>volatile</durability>
+                      <history depth="1">keep_last</history>
+                      <liveliness>automatic</liveliness>
+                    </publisher>
+                  </topic>
+                </qos>
+              </ros>
+            </plugin>
+          </xacro:if>
         </sensor>
-      </xacro:if>
-      <xacro:if value="${gazebo_version == 'gazebo'}">
-        <sensor type="rgbd_camera" name="${name}_frame_sensor">
-          <ignition_frame_id>${name}_optical_frame</ignition_frame_id>
-          <camera>
-            <horizontal_fov>${58.0 * deg_to_rad}</horizontal_fov>
-            <image>
-              <format>R8G8B8</format>
-              <width>320</width>
-              <height>240</height>
-            </image>
-            <clip>
-              <near>0.45</near>
-              <far>10.0</far>
-            </clip>
-            <distortion>
-              <k1>0.0</k1>
-              <k2>0.0</k2>
-              <k3>0.0</k3>
-              <p1>0.0</p1>
-              <p2>0.0</p2>
-            </distortion>
-            <depth_camera>
-              <clip>
-                <near>0.1</near>
-                <far>10</far>
-              </clip>
-            </depth_camera>
-            <noise>
-              <type>gaussian</type>
-              <mean>0</mean>
-              <stddev>0.003</stddev>
-            </noise>
-          </camera>
-          <always_on>1</always_on>
-          <update_rate>10</update_rate>
-          <visualize>0</visualize>
-          <topic>${name}</topic>
-        </sensor>
-      </xacro:if>
     </gazebo>
   </xacro:macro>

Commit message: Revert "Merge branch 'tun/feat/update-sensor-gazebo' into 'humble-devel'"
This reverts merge request !26

File: urdf/camera/structure_sensor.gazebo.xacro (robot description, xacro)
@@ -14,114 +14,101 @@
 <robot xmlns:xacro="http://ros.org/wiki/xacro">
   <xacro:macro name="structure_sensor_rgbd_camera_gazebo" params="name">
-    <xacro:if value="${gazebo_version == 'classic'}">
-      <xacro:property name="camera_type" value="depth"/>
-    </xacro:if>
-    <xacro:if value="${gazebo_version == 'gazebo'}">
-      <xacro:property name="camera_type" value="rgbd_camera"/>
-    </xacro:if>
     <gazebo reference="${name}_link">
       <!-- IR + depth -->
-        <sensor type="${camera_type}" name="${name}_frame_sensor">
-          <always_on>true</always_on>
-          <update_rate>6.0</update_rate>
-          <gz_frame_id>${name}_optical_frame</gz_frame_id>
-          <always_on>1</always_on>
-          <update_rate>10</update_rate>
-          <visualize>0</visualize>
-          <topic>${name}</topic>
-          <camera>
-            <horizontal_fov>${58.0 * deg_to_rad}</horizontal_fov>
-            <image>
-              <format>R8G8B8</format>
-              <width>320</width>
-              <height>240</height>
-            </image>
-            <clip>
-              <near>0.45</near>
-              <far>10.0</far>
-            </clip>
-            <distortion>
-              <k1>0.0</k1>
-              <k2>0.0</k2>
-              <k3>0.0</k3>
-              <p1>0.0</p1>
-              <p2>0.0</p2>
-            </distortion>
-          </camera>
-          <xacro:if value="${gazebo_version == 'classic'}">
-            <plugin name="${name}_ir" filename="libgazebo_ros_camera.so">
-              <camera_name>${name}</camera_name>
-              <frame_name>${name}_optical_frame</frame_name>
-              <max_depth>10.0</max_depth>
-              <ros>
-                <namespace>${namespace}</namespace>
-                <remapping>${name}/image_raw:=${name}/ir/image_raw</remapping>
-                <remapping>${name}/camera_info:=${name}/ir/camera_info</remapping>
-                <remapping>${name}/image_raw/compressed:=${name}/ir/image_raw/compressed</remapping>
-                <remapping>${name}/image_raw/compressedDepth:=${name}/ir/image_raw/compressedDepth</remapping>
-                <remapping>${name}/image_raw/theora:=${name}/ir/image_raw/theora</remapping>
-                <remapping>${name}/points:=${name}/depth/points</remapping>
-                <qos>
-                  <topic name="${name}/ir/image_raw">
-                    <publisher>
-                      <reliability>best_effort</reliability>
-                      <durability>volatile</durability>
-                      <history depth="1">keep_last</history>
-                      <liveliness>automatic</liveliness>
-                    </publisher>
-                  </topic>
-                  <topic name="${name}/ir/image_raw/compressed">
-                    <publisher>
-                      <reliability>best_effort</reliability>
-                      <durability>volatile</durability>
-                      <history depth="1">keep_last</history>
-                      <liveliness>automatic</liveliness>
-                    </publisher>
-                  </topic>
-                  <topic name="${name}/ir/image_raw/compressedDepth">
-                    <publisher>
-                      <reliability>best_effort</reliability>
-                      <durability>volatile</durability>
-                      <history depth="1">keep_last</history>
-                      <liveliness>automatic</liveliness>
-                    </publisher>
-                  </topic>
-                  <topic name="${name}/depth/image_raw">
-                    <publisher>
-                      <reliability>best_effort</reliability>
-                      <durability>volatile</durability>
-                      <history depth="1">keep_last</history>
-                      <liveliness>automatic</liveliness>
-                    </publisher>
-                  </topic>
-                  <topic name="${name}/depth/image_raw/compressed">
-                    <publisher>
-                      <reliability>best_effort</reliability>
-                      <durability>volatile</durability>
-                      <history depth="1">keep_last</history>
-                      <liveliness>automatic</liveliness>
-                    </publisher>
-                  </topic>
-                  <topic name="${name}/depth/image_raw/compressedDepth">
-                    <publisher>
-                      <reliability>best_effort</reliability>
-                      <durability>volatile</durability>
-                      <history depth="1">keep_last</history>
-                      <liveliness>automatic</liveliness>
-                    </publisher>
-                  </topic>
-                  <topic name="${name}/depth/points">
-                    <publisher>
-                      <reliability>best_effort</reliability>
-                      <durability>volatile</durability>
-                      <history depth="1">keep_last</history>
-                      <liveliness>automatic</liveliness>
-                    </publisher>
-                  </topic>
-                </qos>
-              </ros>
-            </plugin>
-          </xacro:if>
-        </sensor>
+      <sensor type="depth" name="${name}_frame_sensor">
+        <always_on>true</always_on>
+        <update_rate>6.0</update_rate>
+        <camera>
+          <horizontal_fov>${58.0 * deg_to_rad}</horizontal_fov>
+          <image>
+            <format>R8G8B8</format>
+            <width>320</width>
+            <height>240</height>
+          </image>
+          <clip>
+            <near>0.45</near>
+            <far>10.0</far>
+          </clip>
+          <distortion>
+            <k1>0.0</k1>
+            <k2>0.0</k2>
+            <k3>0.0</k3>
+            <p1>0.0</p1>
+            <p2>0.0</p2>
+          </distortion>
+        </camera>
+        <plugin name="${name}_ir" filename="libgazebo_ros_camera.so">
+          <camera_name>${name}</camera_name>
+          <frame_name>${name}_optical_frame</frame_name>
+          <max_depth>10.0</max_depth>
+          <ros>
+            <namespace>${namespace}</namespace>
+            <remapping>${name}/image_raw:=${name}/ir/image_raw</remapping>
+            <remapping>${name}/camera_info:=${name}/ir/camera_info</remapping>
+            <remapping>${name}/image_raw/compressed:=${name}/ir/image_raw/compressed</remapping>
+            <remapping>${name}/image_raw/compressedDepth:=${name}/ir/image_raw/compressedDepth</remapping>
+            <remapping>${name}/image_raw/theora:=${name}/ir/image_raw/theora</remapping>
+            <remapping>${name}/points:=${name}/depth/points</remapping>
+            <qos>
+              <topic name="${name}/ir/image_raw">
+                <publisher>
+                  <reliability>best_effort</reliability>
+                  <durability>volatile</durability>
+                  <history depth="1">keep_last</history>
+                  <liveliness>automatic</liveliness>
+                </publisher>
+              </topic>
+              <topic name="${name}/ir/image_raw/compressed">
+                <publisher>
+                  <reliability>best_effort</reliability>
+                  <durability>volatile</durability>
+                  <history depth="1">keep_last</history>
+                  <liveliness>automatic</liveliness>
+                </publisher>
+              </topic>
+              <topic name="${name}/ir/image_raw/compressedDepth">
+                <publisher>
+                  <reliability>best_effort</reliability>
+                  <durability>volatile</durability>
+                  <history depth="1">keep_last</history>
+                  <liveliness>automatic</liveliness>
+                </publisher>
+              </topic>
+              <topic name="${name}/depth/image_raw">
+                <publisher>
+                  <reliability>best_effort</reliability>
+                  <durability>volatile</durability>
+                  <history depth="1">keep_last</history>
+                  <liveliness>automatic</liveliness>
+                </publisher>
+              </topic>
+              <topic name="${name}/depth/image_raw/compressed">
+                <publisher>
+                  <reliability>best_effort</reliability>
+                  <durability>volatile</durability>
+                  <history depth="1">keep_last</history>
+                  <liveliness>automatic</liveliness>
+                </publisher>
+              </topic>
+              <topic name="${name}/depth/image_raw/compressedDepth">
+                <publisher>
+                  <reliability>best_effort</reliability>
+                  <durability>volatile</durability>
+                  <history depth="1">keep_last</history>
+                  <liveliness>automatic</liveliness>
+                </publisher>
+              </topic>
+              <topic name="${name}/depth/points">
+                <publisher>
+                  <reliability>best_effort</reliability>
+                  <durability>volatile</durability>
+                  <history depth="1">keep_last</history>
+                  <liveliness>automatic</liveliness>
+                </publisher>
+              </topic>
+            </qos>
+          </ros>
+        </plugin>
+      </sensor>
     </gazebo>
   </xacro:macro>

File: urdf/camera/structure_sensor.urdf.xacro (robot description, xacro)
@@ -73,5 +73,5 @@
     <link name="${name}_depth_optical_frame"/>
     <!-- extensions -->
-    <xacro:structure_sensor_rgbd_camera_gazebo name="${name}"/>
+    <xacro:structure_sensor_rgbd_camera_gazebo name="${name}" />
   </xacro:macro>
 </robot>

File: urdf/laser/sick_tim571_laser.gazebo.xacro (robot description, xacro)
@@ -27,5 +27,5 @@
               <samples>${818*(max_angle - min_angle)/(270.0 * deg_to_rad)}</samples>
               <resolution>1</resolution>              <!-- not the sensor resolution; just 1 -->
-              <min_angle>${min_angle -1}</min_angle> <!--there is a laserscan detecting ghost obstacle-->
+              <min_angle>${min_angle}</min_angle>
               <max_angle>${max_angle}</max_angle>
             </horizontal>

File: urdf/laser/sick_tim571_laser.urdf.xacro (robot description, xacro)
@@ -42,5 +42,5 @@
     </joint>
     <!-- gazebo extensions -->
-    <xacro:sick_tim571_laser_gazebo name="${name}" ros_topic="${ros_topic}" update_rate="${update_rate}" min_angle="${min_angle}" max_angle="${max_angle}"/>
+    <xacro:sick_tim571_laser_gazebo name="${name}" ros_topic="${ros_topic}" update_rate="${update_rate}" min_angle="${min_angle}" max_angle="${max_angle}" />
   </xacro:macro>
 </robot>
