Commit message: fixing laser

File: urdf/laser/ydlidar_tg30_laser.urdf.xacro (robot description, xacro)
@@ -21,5 +21,5 @@
         <origin xyz="0 0 0" rpy="0 0 0" />
         <geometry>
-          <mesh filename="file://$(find pal_urdf_utils)/meshes/laser/ydlidar.dae"/>
+          <mesh filename="file://$(find pal_urdf_utils)/meshes/laser/YDlidarTG15_30_50.STL"/>
         </geometry>
         <material name="DarkGrey"/>
@@ -28,5 +28,5 @@
         <origin xyz="0 0 0" rpy="0 0 0" />
         <geometry>
-          <mesh filename="file://$(find pal_urdf_utils)/meshes/laser/ydlidar.dae"/>
+          <mesh filename="file://$(find pal_urdf_utils)/meshes/laser/YDlidarTG15_30_50.STL"/>
         </geometry>
       </collision>

Commit message: changing name mesh

File: urdf/laser/ydlidar_tg30_laser.urdf.xacro (robot description, xacro)
@@ -21,5 +21,5 @@
         <origin xyz="0 0 0" rpy="0 0 0" />
         <geometry>
-          <mesh filename="file://$(find pal_urdf_utils)/meshes/laser/YDlidarTG15_30_50.STL"/>
+          <mesh filename="file://$(find pal_urdf_utils)/meshes/laser/ydlidar.stl"/>
         </geometry>
         <material name="DarkGrey"/>
@@ -28,5 +28,5 @@
         <origin xyz="0 0 0" rpy="0 0 0" />
         <geometry>
-          <mesh filename="file://$(find pal_urdf_utils)/meshes/laser/YDlidarTG15_30_50.STL"/>
+          <mesh filename="file://$(find pal_urdf_utils)/meshes/laser/ydlidar.stl"/>
         </geometry>
       </collision>
