Commit message: add gazebo parameter to sick tim 571

File: urdf/laser/sick_tim571_laser.gazebo.xacro (robot description, xacro)
@@ -13,5 +13,9 @@
  -->
 <robot xmlns:xacro="http://ros.org/wiki/xacro">
-  <xacro:macro name="sick_tim571_laser_gazebo" params="name ros_topic update_rate min_angle max_angle">
+  <xacro:macro name="sick_tim571_laser_gazebo" params="name ros_topic update_rate min_angle max_angle gazebo_version">
+    <xacro:property name="gazebo_version" value="$(arg gazebo_version)"/>
+    <xacro:if value="${gazebo_version not in ['classic', 'gazebo']}">
+      <xacro:wrong_gazebo_version/>
+    </xacro:if>
     <gazebo reference="${name}_link">
       <sensor name="${name}" type="gpu_lidar">

File: urdf/laser/sick_tim571_laser.urdf.xacro (robot description, xacro)
@@ -14,5 +14,5 @@
 <robot xmlns:xacro="http://ros.org/wiki/xacro">
   <xacro:include filename="$(find pal_urdf_utils)/urdf/laser/sick_tim571_laser.gazebo.xacro" />
-  <xacro:macro name="sick_tim571_laser" params="name parent *origin ros_topic update_rate min_angle max_angle">
+  <xacro:macro name="sick_tim571_laser" params="name parent *origin ros_topic update_rate min_angle max_angle gazebo_version:=classic">
     <link name="${name}_link" type="laser">
       <inertial>
@@ -42,5 +42,5 @@
     </joint>
     <!-- gazebo extensions -->
-    <xacro:sick_tim571_laser_gazebo name="${name}" ros_topic="${ros_topic}" update_rate="${update_rate}" min_angle="${min_angle}" max_angle="${max_angle}" />
+    <xacro:sick_tim571_laser_gazebo name="${name}" ros_topic="${ros_topic}" update_rate="${update_rate}" min_angle="${min_angle}" max_angle="${max_angle}" gazebo_version="${gazebo_version}"/>
   </xacro:macro>
 </robot>

Commit message: remove gazebo version check property

File: urdf/laser/sick_tim571_laser.gazebo.xacro (robot description, xacro)
@@ -14,8 +14,4 @@
 <robot xmlns:xacro="http://ros.org/wiki/xacro">
   <xacro:macro name="sick_tim571_laser_gazebo" params="name ros_topic update_rate min_angle max_angle">
-    <xacro:property name="gazebo_version" value="$(arg gazebo_version)"/>
-    <xacro:if value="${gazebo_version not in ['classic', 'gazebo']}">
-      <xacro:wrong_gazebo_version/>
-    </xacro:if>
     <gazebo reference="${name}_link">
       <sensor name="${name}" type="gpu_lidar">
